Commit message: Update camera to RGBD in urdf

File: my_robot/urdf/my_robot.xacro (robot description, xacro)
@@ -16,7 +16,7 @@
       <origin xyz="0.0 0 0" rpy=" 0 0 0"/>
       <inertia
-          ixx="0.06" ixy="0" ixz="0"
-          iyy="0.06" iyz="0"
-          izz="0.06"
+          ixx="0.03" ixy="0" ixz="0"
+          iyy="0.03" iyz="0"
+          izz="0.03"
       />
     </inertial>
@@ -25,31 +25,5 @@
       <geometry>
         <box size=".2 .1 .06"/>
-      </geometry><link name="camera">
-    <collision>
-      <origin xyz="0 0 0" rpy="0 0 0"/>
-      <geometry>
-        <box size="${cameraSize} ${cameraSize} ${cameraSize}"/>
       </geometry>
-    </collision>
-    <visual>
-      <origin xyz="0 0 0" rpy="0 0 0"/>
-      <geometry>
-        <box size="${cameraSize} ${cameraSize} ${cameraSize}"/>
-      </geometry>
-      <material name="green"/>
-    </visual>
-    <inertial>
-      <mass value="${cameraMass}" />
-      <origin xyz="0 0 0" rpy="0 0 0"/>
-      <box_inertia m="${cameraMass}" x="${cameraSize}" y="${cameraSize}" z="${cameraSize}" />
-      <inertia ixx="1e-6" ixy="0" ixz="0" iyy="1e-6" iyz="0" izz="1e-6" />
-    </inertial>
-  </link>
-  <joint name="camera_joint" type="fixed">
-    <axis xyz="0 1 0" />
-    <origin xyz=".1 0 0" rpy="0 0 0"/>
-    <parent link="chassis"/>
-    <child link="camera"/>
-  </joint>
     </collision>
     <visual name='chassis_visual'>
@@ -102,7 +76,7 @@
       <mass value="0.5"/>
       <inertia
-        ixx=".05" ixy="0.0" ixz="0.0"
-        iyy=".05" iyz="0.0"
-        izz=".05"/>
+        ixx=".01" ixy="0.0" ixz="0.0"
+        iyy=".01" iyz="0.0"
+        izz=".01"/>
     </inertial>
   </link>
@@ -125,7 +99,7 @@
       <mass value="0.5"/>
       <inertia
-        ixx=".05" ixy="0.0" ixz="0.0"
-        iyy=".05" iyz="0.0"
-        izz=".05"/>
+        ixx=".01" ixy="0.0" ixz="0.0"
+        iyy=".01" iyz="0.0"
+        izz=".01"/>
     </inertial>
   </link>
@@ -175,4 +149,11 @@
     <child link="camera"/>
   </joint>
+  <joint name="camera_optical_joint" type="fixed">
+    <origin xyz="0 0 0" rpy="-1.5707 0 -1.5707"/>
+    <parent link="camera"/>
+    <child link="camera_link_optical"/>
+  </joint>
+  <link name="camera_link_optical">
+  </link>
  <joint name="hokuyo_joint" type="fixed">
     <axis xyz="0 1 0" />
